File: kuttyPy/hardware/microhope.sch (KiCad schematic (older format))
At the start: 30 parts, among them J1 USB, P1 CONN_10, P2 TST, P3 CONN_10, P4 CONN_10, P5 CONN_10, P6 CONN_5, P7 TST, SW1 RESET, U1 ATMEGA32, U2 CH340G, X1 8MHz, X2 12M

Commit message: removed yet another personalized file reference
Parts:
- D1, D2: symbol LED -> LED-RESCUE-microhope
Changed lines of the file:
@@
 EESchema Schematic File Version 2
+LIBS:microhope-rescue
 LIBS:power
 LIBS:device
@@
 LIBS:memory
 LIBS:xilinx
-LIBS:microcontrollers
-LIBS:dsp
-LIBS:microchip
-LIBS:analog_switches
-LIBS:motorola
-LIBS:texas
-LIBS:intel
-LIBS:audio
-LIBS:interface
-LIBS:digital-audio
-LIBS:philips
-LIBS:display
-LIBS:cypress
-LIBS:siliconi
-LIBS:opto
-LIBS:atmel
-LIBS:contrib
-LIBS:valves
-LIBS:proto1
 LIBS:microhope-cache
 EELAYER 25 0
@@
 $EndComp
 $Comp
-L LED D2
+L LED-RESCUE-microhope D2
 U 1 1 52786D0B
 P 3750 4700
@@
 $EndComp
 $Comp
-L LED D1
+L LED-RESCUE-microhope D1
 U 1 1 527880C3
 P 4750 1000
